Commit message: Fix urdf dimensions

File: urdf/robot.urdf (robot description, URDF)
Before this commit: robot robo_pet, 9 links, 8 joints
Links:
- link base_link: geometry visual box size=0.3300 0.3310 0.1260

Commit message: lidar

File: urdf/robot.urdf (robot description, URDF)
Before this commit: robot robo_pet, 9 links, 8 joints
Links:
- added link laser
Joints:
- added joint base_to_laser: type fixed, parent base_link, child laser, origin xyz=0.0000 0.0000 0.3000 rpy=0.0000 0.0000 0.0000

Commit message: fix lidar mount offset

File: urdf/robot.urdf (robot description, URDF)
Before this commit: robot robo_pet, 10 links, 9 joints
Joints:
- joint base_to_laser: origin xyz=0.0000 0.0000 0.3000 rpy=0.0000 0.0000 0.0000 -> xyz=-0.0820 0.0000 0.2030 rpy=0.0000 0.0000 0.0000

Commit message: More accurate movement

File: urdf/robot.urdf (robot description, URDF)
Before this commit: robot robo_pet, 10 links, 9 joints
Links:
- link left_wheel: geometry visual cylinder length=0.0300 radius=0.0501
- link right_wheel: geometry visual cylinder length=0.0300 radius=0.0501
Joints:
- joint base_to_left_wheel: origin xyz=0.0000 0.1530 0.0480 rpy=0.0000 0.0000 0.0000 -> xyz=0.0000 0.1530 0.0501 rpy=0.0000 0.0000 0.0000
- joint base_to_right_wheel: origin xyz=0.0000 -0.1530 0.0480 rpy=0.0000 0.0000 0.0000 -> xyz=0.0000 -0.1530 0.0501 rpy=0.0000 0.0000 0.0000

Commit message: timed turns

File: urdf/robot.urdf (robot description, URDF)
Before this commit: robot robo_pet, 10 links, 9 joints
Joints:
- joint base_to_left_wheel: origin xyz=0.0000 0.1530 0.0501 rpy=0.0000 0.0000 0.0000 -> xyz=0.0000 0.1600 0.0501 rpy=0.0000 0.0000 0.0000
- joint base_to_right_wheel: origin xyz=0.0000 -0.1530 0.0501 rpy=0.0000 0.0000 0.0000 -> xyz=0.0000 -0.1600 0.0501 rpy=0.0000 0.0000 0.0000
