Commit message: Robot geometry: measured on the robot, 2026-10-26
Bumper face 51 mm ahead of the axle (was 55). Footprint front 0.060 (cliff
tips), rear -0.284 (caster swung fully back, was -0.266), half width 0.166.
Forward ToF chips at x -0.061 / y +-0.112 and centre x +0.0115, cliff ToFs at
x 0.060, IMU mount added at its measured spot. Nav2 footprint follows.

Co-Authored-By: Claude Opus 5.5 <noreply@anthropic.com>

File: urdf/robot.urdf (robot description, URDF)
Before this commit: robot robo_pet, 10 links, 9 joints
Links:
- link base_link: geometry visual box size=0.3440 0.3320 0.1260
Joints:
- joint base_to_cliff_left: origin xyz=0.0640 0.1280 0.0670 rpy=0.0000 0.6109 0.0000 -> xyz=0.0600 0.1280 0.0670 rpy=0.0000 0.6109 0.0000
- joint base_to_cliff_right: origin xyz=0.0640 -0.1280 0.0670 rpy=0.0000 0.6109 0.0000 -> xyz=0.0600 -0.1280 0.0670 rpy=0.0000 0.6109 0.0000
- joint base_to_forward_center: origin xyz=0.0100 0.0000 0.1100 rpy=0.0000 0.0000 0.0000 -> xyz=0.0115 0.0000 0.1100 rpy=0.0000 0.0000 0.0000
- joint base_to_forward_left: origin xyz=-0.0630 0.1100 0.1260 rpy=0.0000 0.0000 0.0000 -> xyz=-0.0610 0.1120 0.1260 rpy=0.0000 0.0000 0.0000
- joint base_to_forward_right: origin xyz=-0.0630 -0.1100 0.1260 rpy=0.0000 0.0000 0.0000 -> xyz=-0.0610 -0.1120 0.1260 rpy=0.0000 0.0000 0.0000
- joint base_to_imu_link: origin xyz=0.0000 0.0000 0.0000 rpy=0.0000 0.0000 0.0000 -> xyz=-0.1278 0.1120 0.1240 rpy=0.0000 0.0000 0.0000
- joint base_to_laser: origin xyz=-0.0820 0.0000 0.2030 rpy=0.0000 0.0000 0.0000 -> xyz=-0.0820 0.0000 0.1960 rpy=0.0000 0.0000 0.0000

Commit message: Robot geometry: side ToF height and leftover old numbers
Side forward ToF chips sit at the board centre, 124 mm up (was 126). The
dimensions doc, forward ToF doc and lidar plan now agree with the measured
footprint and sensor positions.

Co-Authored-By: Claude Opus 5.5 <noreply@anthropic.com>

File: urdf/robot.urdf (robot description, URDF)
Before this commit: robot robo_pet, 10 links, 9 joints
Links:
- link base_link: geometry visual box size=0.3440 0.3320 0.1240
Joints:
- joint base_to_forward_left: origin xyz=-0.0610 0.1120 0.1260 rpy=0.0000 0.0000 0.0000 -> xyz=-0.0610 0.1120 0.1240 rpy=0.0000 0.0000 0.0000
- joint base_to_forward_right: origin xyz=-0.0610 -0.1120 0.1260 rpy=0.0000 0.0000 0.0000 -> xyz=-0.0610 -0.1120 0.1240 rpy=0.0000 0.0000 0.0000
